Commit message: Split the <gazebo> tags into a new file. Changed some inertia properties. Added IMU

File: src/mmtr_description/urdf/mmtr_core.xacro (robot description, xacro)
@@ -3,9 +3,9 @@
 	<plugin name="gazebo_ros_paths" filename="libgazebo_ros_paths_plugin.so" />
 	<xacro:property name="mesh_dir" value="file://$(find mmtr_description)/meshes/" />
-  	<!-- <xacro:include filename="$(find mmtr_description)/urdf/mmtr_ros_2_control.xacro" /> -->
-	<xacro:property name="flipper_mass" value="0.375" />
+	<!-- <xacro:include filename="$(find mmtr_description)/urdf/mmtr_ros_2_control.xacro" /> -->
+	<xacro:include filename="mmtr_gazebo.xacro" />
 	<xacro:include filename="inertial_macros.xacro" />
 	<!-- ********** MACROS ********** -->
-	<xacro:property name="mass" value="1.5"> </xacro:property>
+	<xacro:property name="mass" value="1.5" />
 	<xacro:property name="flipper_mass" value="0.375" />
 	<xacro:property name="flipper_length" value="0.12932" />
@@ -13,5 +13,5 @@
 	<xacro:property name="flipper_radius" value="0.06958" />
 	<!-- ********** MACROS ********** -->
-	<!-- ********** BASE LINK ********** -->
+	<!-- ********** BASE FOOTPRINT ********** -->
 	<link name="base_footprint" />
 	<joint name="chassis_joint" type="fixed">
@@ -20,21 +20,18 @@
 		<origin xyz="0.0 0.0 0.0" rpy="0.0 0.0 0.0" />
 	</joint>
+	<!-- ********** BASE FOOTPRINT ********** -->
 	<!-- ********** BASE LINK ********** -->
-	<!-- ********** CHASSIS LINK ********** -->
 	<link name="base_link">
-		<xacro:inertial_box mass="1" x="0.25" y="0.175" z="0.06">
-    <origin xyz="-4.4639E-06 -1.1907E-06 -0.0036869" rpy="0 0 0" />
-		</xacro:inertial_box>
-<!-- <inertial>
-    <origin xyz="-4.4639E-06 -1.1907E-06 -0.0036869" rpy="0 0 0" />
-    <mass value="3.0" />
-    <inertia
-        ixx="0.0055239"
-        ixy="9.7788E-07"
-        ixz="1.5028E-07"
-        iyy="0.0215439"
-        iyz="2.2009E-07"
-        izz="0.0251589" />
-</inertial> -->
+		<inertial>
+			<origin xyz="-4.4639E-06 -1.1907E-06 -0.0036869" rpy="0 0 0" />
+			<mass value="3.0" />
+			<inertia
+				ixx="0.0055239"
+				ixy="9.7788E-07"
+				ixz="1.5028E-07"
+				iyy="0.0215439"
+				iyz="2.2009E-07"
+				izz="0.0251589" />
+		</inertial>
 		<visual>
 			<origin xyz="0 0 0" rpy="0 0 0" />
@@ -62,31 +59,18 @@
 		</collision>
 	</link>
-	<gazebo reference="base_link">
-		<self_collide>1</self_collide>
-		<mu1>100.0</mu1>
-		<mu2>100.0</mu2>
-		<kp value="10000000.0" />
-		<kd value="1.0" />
-		<fdir1 value="0 1 0" />
-		<maxContacts>2</maxContacts>
-	</gazebo>
 	<!-- ********** CHASSIS LINK ********** -->
 	<!-- ********** LEFT FLIPPER LINK ********** -->
-	<link
-		name="front_flipper_left">
-				<xacro:inertial_box mass="${flipper_mass}" x="0.139577" y="0.045" z="0.06958">
-    <origin xyz="0.039257 -0.01033 -0.00014149" rpy="0 0 0" />
-		</xacro:inertial_box>
-<!-- <inertial>
-    <origin xyz="0.039257 -0.01033 -0.00014149" rpy="0 0 0" />
-    <mass value="2.0" />
-    <inertia
-        ixx="0.0008184"
-        ixy="-4.6196E-05"
-        ixz="4.2342E-07"
-        iyy="0.0029431"
-        iyz="3.2476E-07"
-        izz="0.00228085" />
-</inertial> -->
+	<link name="front_flipper_left">
+		<inertial>
+			<origin xyz="0.039257 -0.01033 -0.00014149" rpy="0 0 0" />
+			<mass value="2.0" />
+			<inertia
+				ixx="0.0008184"
+				ixy="-4.6196E-05"
+				ixz="4.2342E-07"
+				iyy="0.0029431"
+				iyz="3.2476E-07"
+				izz="0.00228085" />
+		</inertial>
 		<visual>
 			<origin xyz="0 0 0" rpy="0 0 0" />
@@ -122,31 +106,18 @@
 		<limit lower="-4" upper="4" effort="10.96" velocity="10.0" />
 	</joint>
-	<gazebo reference="front_flipper_left">
-		<mu1>100.0</mu1>
-		<mu2>100.0</mu2>
-		<kp value="10000000.0" />
-		<kd value="1.0" />
-		<fdir1 value="0 1 0" />
-		<gravity>1</gravity>
-		<maxContacts>2</maxContacts>
-		<material>Gazebo/DarkGrey</material>
-	</gazebo>
 	<!-- ********** LEFT FLIPPER LINK ********** -->
 	<!-- ********** RIGHT FLIPPER LINK ********** -->
 	<link name="front_flipper_right">
-<!-- <inertial>
-    <origin xyz="0.039266 0.01033 0.00013504" rpy="0 0 0" />
-    <mass value="2.0" />
-    <inertia
-        ixx="0.0008184"
-        ixy="0.000046196"
-        ixz="-0.00000042342"
-        iyy="0.0029431"
-        iyz="0.00000032476"
-        izz="0.00228085" />
-</inertial> -->
-		<xacro:inertial_box mass="${flipper_mass}" x="0.139577" y="0.045" z="0.06958">
-    <origin xyz="0.039266 0.01033 0.00013504" rpy="0 0 0" />
-		</xacro:inertial_box>
+		<inertial>
+			<origin xyz="0.039266 0.01033 0.00013504" rpy="0 0 0" />
+			<mass value="2.0" />
+			<inertia
+				ixx="0.0008184"
+				ixy="0.000046196"
+				ixz="-0.00000042342"
+				iyy="0.0029431"
+				iyz="0.00000032476"
+				izz="0.00228085" />
+		</inertial>
 		<visual>
 			<origin xyz="0 0 0" rpy="0 0 0" />
@@ -181,31 +152,18 @@
 		<limit lower="-4" upper="4" effort="1.96" velocity="1.0" />
 	</joint>
-	<gazebo reference="front_flipper_right">
-		<mu1>100.0</mu1>
-		<mu2>100.0</mu2>
-		<kp value="10000000.0" />
-		<kd value="1.0" />
-		<fdir1 value="0 1 0" />
-		<gravity>1</gravity>
-		<maxContacts>2</maxContacts>
-		<material>Gazebo/DarkGrey</material>
-	</gazebo>
 	<!-- ********** RIGHT FLIPPER LINK ********** -->
 	<!-- ********** REAR RIGHT FLIPPER LINK ********** -->
 	<link name="rear_flipper_right">
-		<!-- <inertial>
+		<inertial>
 			<origin xyz="-0.039256 0.01033 -0.0001417" rpy="0 0 0" />
-    <mass value="2.0" />
-    <inertia
-        ixx="0.0008184"
-        ixy="0.000046196"
-        ixz="-0.00000042342"
-        iyy="0.0029431"
-        iyz="0.00000032476"
-        izz="0.00228085" />
-</inertial> -->
-		<xacro:inertial_box mass="${flipper_mass}" x="0.139577" y="0.045" z="0.06958">
-			<origin xyz="-0.039256 0.01033 -0.0001417" rpy="0 0 0" />
-		</xacro:inertial_box>
+			<mass value="2.0" />
+			<inertia
+				ixx="0.0008184"
+				ixy="0.000046196"
+				ixz="-0.00000042342"
+				iyy="0.0029431"
+				iyz="0.00000032476"
+				izz="0.00228085" />
+		</inertial>
 		<visual>
 			<origin xyz="0 0 0" rpy="0 0 0" />
@@ -240,31 +198,18 @@
 		<limit lower="-4" upper="4" effort="1.96" velocity="1.0" />
 	</joint>
-	<gazebo reference="rear_flipper_right">
-		<mu1>100.0</mu1>
-		<mu2>100.0</mu2>
-		<kp value="10000000.0" />
-		<kd value="1.0" />
-		<fdir1 value="0 1 0" />
-		<gravity>1</gravity>
-		<maxContacts>2</maxContacts>
-		<material>Gazebo/DarkGrey</material>
-	</gazebo>
 	<!-- ********** REAR RIGHT FLIPPER LINK ********** -->
 	<!-- ********** REAR LEFT FLIPPER LINK ********** -->
 	<link name="rear_flipper_left">
-		<!-- <inertial>
+		<inertial>
 			<origin xyz="-0.039262 -0.01033 0.00013791" rpy="0 0 0" />
-    <mass value="2.0" />
-    <inertia
-        ixx="0.0008184"
-        ixy="0.000046196"
-        ixz="-0.00000042342"
-        iyy="0.0029431"
-        iyz="0.00000032476"
-        izz="0.00228085" />
-</inertial> -->
-		<xacro:inertial_box mass="${flipper_mass}" x="0.139577" y="0.045" z="0.06958">
-			<origin xyz="-0.039262 -0.01033 0.00013791" rpy="0 0 0" />
-		</xacro:inertial_box>
+			<mass value="2.0" />
+			<inertia
+				ixx="0.0008184"
+				ixy="0.000046196"
+				ixz="-0.00000042342"
+				iyy="0.0029431"
+				iyz="0.00000032476"
+				izz="0.00228085" />
+		</inertial>
 		<visual>
 			<origin xyz="0 0 0" rpy="0 0 0" />
@@ -299,17 +244,39 @@
 		<limit lower="-4" upper="4" effort="1.96" velocity="1.0" />
 	</joint>
-	<gazebo reference="rear_flipper_left">
-		<mu1>100.0</mu1>
-		<mu2>100.0</mu2>
-		<kp value="10000000.0" />
-		<kd value="1.0" />
-		<fdir1 value="0 1 0" />
-		<gravity>1</gravity>
-		<maxContacts>2</maxContacts>
-		<material>Gazebo/DarkGrey</material>
-	</gazebo>
 	<!-- ********** REAR LEFT FLIPPER LINK ********** -->
-  <!-- Transmission for ros2_control -->
-  <!-- <transmission name="front_left_flipper_transmission">
+	<!-- ********** IMU LINK ********** -->
+	<link name="imu_link">
+		<inertial>
+			<origin xyz="-0.00552433659106688 0.000168210391520346 0.000514000497342681" rpy="0 0 0" />
+			<mass value="0.0005" />
+			<inertia
+				ixx="4.05951542e-08"
+				ixy="0.0"
+				ixz="0.0"
+				iyy="1.20848833e-08"
+				iyz="0.0"
+				izz="5.21424042e-08" />
+		</inertial>
+		<visual>
+			<origin xyz="0 0 0" rpy="0 0 0" />
+			<geometry>
+				<box size="0.01684 0.03111 0.00254" />
+			</geometry>
+		</visual>
+		<collision>
+			<origin xyz="0 0 0" rpy="0 0 0" />
+			<geometry>
+				<box size="0.01684 0.03111 0.00254" />
+			</geometry>
+		</collision>
+	</link>
+	<joint name="imu_joint" type="fixed">
+		<parent link="base_link" />
+		<child link="imu_link" />
+		<origin xyz="0.0 0.0 0.015" rpy="0.0 0.0 0.0" />
+		<axis xyz="0 0 0" />
+	</joint>
+	<!-- Transmission for ros2_control -->
+	<!-- <transmission name="front_left_flipper_transmission">
     <type>transmission_interface/SimpleTransmission</type>
     <actuator name="front_left_flipper_motor"/>
@@ -317,8 +284,8 @@
     <mechanicalReduction>1</mechanicalReduction>
   </transmission> -->
-  <!-- ros2_control configuration -->
-	 <ros2_control name="GazeboSystem" type="system">
+	<!-- ros2_control configuration -->
+	<ros2_control name="GazeboSystem" type="system">
 		<hardware>
-            <plugin>gz_ros2_control/GazeboSimSystem</plugin>
+			<plugin>gz_ros2_control/GazeboSimSystem</plugin>
 		</hardware>
 		<joint name="front_left_flipper_joint">
@@ -329,11 +296,4 @@
 			<state_interface name="position" />
 		</joint>
-  </ros2_control>
-	<gazebo>
-		<plugin name="gz_ros2_control::GazeboSimROS2ControlPlugin" filename="libgz_ros2_control-system.so">
-			<robot_param>robot_description</robot_param>
-			<robot_param_node>robot_state_publisher</robot_param_node>
-			<parameters>$(find mmtr_description)/config/flipper_controller.yaml</parameters>
-		</plugin>
-	</gazebo>
+	</ros2_control>
 </robot>

Commit message: Added a laser link

File: src/mmtr_description/urdf/mmtr_core.xacro (robot description, xacro)
@@ -275,4 +275,32 @@
 		<child link="imu_link" />
 		<origin xyz="0.0 0.0 0.015" rpy="0.0 0.0 0.0" />
+		<axis xyz="0 0 0" />
+	</joint>
+	<link name="laser_link">
+		<inertial>
+			<origin xyz="-0.011945780406062 -0.000381929217680526 -0.0170649378129477" rpy="0 0 0" />
+			<mass value="0.073084435549317" />
+			<inertia ixx="1.96074931730795E-05" ixy="-3.62091076640009E-07"
+				ixz="4.28230084046735E-07"
+				iyy="2.40983835136327E-05" iyz="1.50180909250652E-08"
+				izz="4.14184164228595E-05" />
+		</inertial>
+		<visual>
+			<origin xyz="0 0 0" rpy="0 0 0" />
+			<geometry>
+				<box size="0.01684 0.03111 0.00254" />
+			</geometry>
+		</visual>
+		<collision>
+			<origin xyz="0 0 0" rpy="0 0 0" />
+			<geometry>
+				<box size="0.01684 0.03111 0.00254" />
+			</geometry>
+		</collision>
+	</link>
+	<joint name="laser_joint" type="fixed">
+		<origin xyz="-0.0050526 -0.0023221 0.1208" rpy="0 0 3.14" />
+		<parent link="base_link" />
+		<child link="laser_link" />
 		<axis xyz="0 0 0" />
 	</joint>
