Commit message: Formatted to use more macros for changing sensor noise easily

File: src/mmtr_description/urdf/mmtr_gazebo.xacro (robot description, xacro)
@@ -1,4 +1,46 @@
 <?xml version="1.0" encoding="utf-8"?>
 <robot xmlns:xacro="http://www.ros.org/wiki/xacro" name="mmtr">
+    <xacro:macro name="imu_linear_noise">
+        <mean>${imu_linear_mean}</mean>
+        <stddev>${imu_linear_stddev}</stddev>
+        <bias_mean>${imu_linear_bias_mean}</bias_mean>
+        <bias_stddev>${imu_linear_bias_stddev}</bias_stddev>
+        <dynamic_bias_stddev>${imu_linear_dynamic_bias_stddev}</dynamic_bias_stddev>
+        <dynamic_bias_correlation_time>${imu_linear_dynamic_bias_correlation_time}</dynamic_bias_correlation_time>
+    </xacro:macro>
+    <xacro:macro name="imu_angular_noise">
+        <mean>${imu_angular_mean}</mean>
+        <stddev>${imu_angular_stddev}</stddev>
+        <bias_mean>${imu_angular_bias_mean}</bias_mean>
+        <bias_stddev>${imu_angular_bias_stddev}</bias_stddev>
+        <dynamic_bias_stddev>${imu_angular_dynamic_bias_stddev}</dynamic_bias_stddev>
+        <dynamic_bias_correlation_time>${imu_angular_dynamic_bias_correlation_time}</dynamic_bias_correlation_time>
+    </xacro:macro>
+    <xacro:macro name="mag_noise">
+        <mean>${mag_mean}</mean>
+        <stddev>${mag_stddev}</stddev>
+        <bias_mean>${mag_bias_mean}</bias_mean>
+        <bias_stddev>${mag_bias_stddev}</bias_stddev>
+        <dynamic_bias_stddev>${mag_dynamic_bias_stddev}</dynamic_bias_stddev>
+        <dynamic_bias_correlation_time>${mag_dynamic_bias_correlation_time}</dynamic_bias_correlation_time>
+    </xacro:macro>
+    <xacro:property name="imu_angular_mean" value="0.0" />
+    <xacro:property name="imu_angular_stddev" value="0.00262" />
+    <xacro:property name="imu_angular_bias_mean" value="0.00" />
+    <xacro:property name="imu_angular_bias_stddev" value="0.0087" />
+    <xacro:property name="imu_angular_dynamic_bias_stddev" value="1.0e-6" />
+    <xacro:property name="imu_angular_dynamic_bias_correlation_time" value="600" />
+    <xacro:property name="imu_linear_mean" value="0.0" />
+    <xacro:property name="imu_linear_stddev" value="0.0226" />
+    <xacro:property name="imu_linear_bias_mean" value="0.00" />
+    <xacro:property name="imu_linear_bias_stddev" value="0.147" />
+    <xacro:property name="imu_linear_dynamic_bias_stddev" value="2.0e-3" />
+    <xacro:property name="imu_linear_dynamic_bias_correlation_time" value="600" />
+    <xacro:property name="mag_mean" value="0.0" />
+    <xacro:property name="mag_bias_mean" value="0.0" />
+    <xacro:property name="mag_stddev" value="4.0e-7" />
+    <xacro:property name="mag_bias_stddev" value="5.0e-6" />
+    <xacro:property name="mag_dynamic_bias_stddev" value="5.8e-8" />
+    <xacro:property name="mag_dynamic_bias_correlation_time" value="600" />
     <gazebo reference="base_link">
         <self_collide>1</self_collide>
@@ -96,36 +138,15 @@
                     <x>
                         <noise type="gaussian">
-                            <mean>0.0</mean>
-                            <stddev>0.00262</stddev>
-                            <bias_mean>0.0</bias_mean>
-                            <bias_stddev>0.0087</bias_stddev>
-                            <!-- Easy mode -->
-                            <dynamic_bias_stddev>1.0e-6</dynamic_bias_stddev>
-                            <!-- <dynamic_bias_stddev>2.80e-6</dynamic_bias_stddev> -->
-                            <dynamic_bias_correlation_time>600.0</dynamic_bias_correlation_time>
+                            <xacro:imu_angular_noise/>
                         </noise>
                     </x>
                     <y>
                         <noise type="gaussian">
-                            <mean>0.0</mean>
-                            <stddev>0.00262</stddev>
-                            <bias_mean>0.0</bias_mean>
-                            <bias_stddev>0.0087</bias_stddev>
-                            <!-- Easy mode -->
-                            <dynamic_bias_stddev>1.0e-6</dynamic_bias_stddev>
-                            <!-- <dynamic_bias_stddev>2.80e-6</dynamic_bias_stddev> -->
-                            <dynamic_bias_correlation_time>600.0</dynamic_bias_correlation_time>
+                            <xacro:imu_angular_noise/>
                         </noise>
                     </y>
                     <z>
                         <noise type="gaussian">
-                            <mean>0.0</mean>
-                            <stddev>0.00262</stddev>
-                            <bias_mean>0.0</bias_mean>
-                            <bias_stddev>0.0087</bias_stddev>
-                            <!-- Easy mode -->
-                            <dynamic_bias_stddev>1.0e-6</dynamic_bias_stddev>
-                            <!-- <dynamic_bias_stddev>2.80e-6</dynamic_bias_stddev> -->
-                            <dynamic_bias_correlation_time>600.0</dynamic_bias_correlation_time>
+                            <xacro:imu_angular_noise/>
                         </noise>
                     </z>
@@ -134,36 +155,15 @@
                     <x>
                         <noise type="gaussian">
-                            <mean>0.0</mean>
-                            <stddev>0.0226</stddev>
-                            <bias_mean>0.0</bias_mean>
-                            <bias_stddev>0.147</bias_stddev>
-                            <!-- Easy Mode -->
-                            <dynamic_bias_stddev>2.0e-3</dynamic_bias_stddev>
-                            <!-- <dynamic_bias_stddev>5.66e-3</dynamic_bias_stddev> -->
-                            <dynamic_bias_correlation_time>600.0</dynamic_bias_correlation_time>
+                            <xacro:imu_linear_noise/>
                         </noise>
                     </x>
                     <y>
                         <noise type="gaussian">
-                            <mean>0.0</mean>
-                            <stddev>0.0226</stddev>
-                            <bias_mean>0.0</bias_mean>
-                            <bias_stddev>0.147</bias_stddev>
-                            <!-- Easy Mode -->
-                            <dynamic_bias_stddev>2.0e-3</dynamic_bias_stddev>
-                            <!-- <dynamic_bias_stddev>5.66e-3</dynamic_bias_stddev> -->
-                            <dynamic_bias_correlation_time>600.0</dynamic_bias_correlation_time>
+                            <xacro:imu_linear_noise/>
                         </noise>
                     </y>
                     <z>
                         <noise type="gaussian">
-                            <mean>0.0</mean>
-                            <stddev>0.0226</stddev>
-                            <bias_mean>0.0</bias_mean>
-                            <bias_stddev>0.147</bias_stddev>
-                            <!-- Easy Mode -->
-                            <dynamic_bias_stddev>2.0e-3</dynamic_bias_stddev>
-                            <!-- <dynamic_bias_stddev>5.66e-3</dynamic_bias_stddev> -->
-                            <dynamic_bias_correlation_time>600.0</dynamic_bias_correlation_time>
+                            <xacro:imu_linear_noise/>
                         </noise>
                     </z>
@@ -183,45 +183,15 @@
             <x>
                 <noise type="gaussian">
-                    <mean>0.0</mean>
-                    <!-- Easy Mode -->
-                    <stddev>4.0e-7</stddev>
-                    <bias_stddev>5.0e-6</bias_stddev>
-                    <dynamic_bias_stddev>5.8e-8</dynamic_bias_stddev>
-                    <dynamic_bias_correlation_time>600.0</dynamic_bias_correlation_time>
-                    <!-- <stddev>1.0e-6</stddev> -->
-                    <!-- <bias_mean>0.0</bias_mean>
-                    <bias_stddev>5.0e-6</bias_stddev>
-                    <dynamic_bias_stddev>5.8e-8</dynamic_bias_stddev>
-                    <dynamic_bias_correlation_time>600.0</dynamic_bias_correlation_time> -->
+                    <xacro:mag_noise/>
                 </noise>
             </x>
             <y>
                 <noise type="gaussian">
-                    <mean>0.0</mean>
-                    <!-- Easy Mode -->
-                    <stddev>4.0e-7</stddev>
-                    <bias_stddev>5.0e-6</bias_stddev>
-                    <dynamic_bias_stddev>5.8e-8</dynamic_bias_stddev>
-                    <dynamic_bias_correlation_time>600.0</dynamic_bias_correlation_time>
-                    <!-- <stddev>1.0e-6</stddev>
-                    <bias_mean>0.0</bias_mean>
-                    <bias_stddev>5.0e-6</bias_stddev>
-                    <dynamic_bias_stddev>5.8e-8</dynamic_bias_stddev>
-                    <dynamic_bias_correlation_time>600.0</dynamic_bias_correlation_time> -->
+                    <xacro:mag_noise/>
                 </noise>
             </y>
             <z>
                 <noise type="gaussian">
-                    <mean>0.0</mean>
-                    <!-- Easy Mode -->
-                    <stddev>4.0e-7</stddev>
-                    <bias_stddev>5.0e-6</bias_stddev>
-                    <dynamic_bias_stddev>5.8e-8</dynamic_bias_stddev>
-                    <dynamic_bias_correlation_time>600.0</dynamic_bias_correlation_time>
-                    <!-- <stddev>1.0e-6</stddev>
-                    <bias_mean>0.0</bias_mean>
-                    <bias_stddev>5.0e-6</bias_stddev>
-                    <dynamic_bias_stddev>5.8e-8</dynamic_bias_stddev>
-                    <dynamic_bias_correlation_time>600.0</dynamic_bias_correlation_time> -->
+                    <xacro:mag_noise/>
                 </noise>
             </z>
